File: hardware/Esp32Tap/kicad/Esp32Tap.kicad_sch (KiCad schematic)
At the start: 50 parts, among them J1 RJ45_Console_54602-908LF, J2 RJ45_Motor_54602-908LF, J3 USB-C_HRO_TYPE-C-31-M-12, K1 G6K-2F-Y-TR DC3, Q1 S8050, SW1 KMR2-EN, SW2 KMR2-BOOT, U1 ESP32-S3-WROOM-1-N8, U2 TPS54202DDCR, U3 USBLC6-2SC6

Commit message: feat(hardware): Esp32Tap order-ready — board-level sim validated, GO verdict
Iterate-until-confident round: applied the validation LED fixes at the
generator source (R11 1k->330R for a visible status LED, R12 2k->1k power
LED) and regenerated the full fab chain (schematic, board, gerbers, BOM,
CPL). ERC/DRC 0 violations; gerber zip re-exported byte-identical to
kicad/gerbers/.

Board-level SPICE (ngspice in Docker) across power / signal-integrity /
relay-transient tracks — all pass with margin: buck input overdamped no
overshoot, EN divider no chatter on a noisy rail, 3.3V droop 27.8mV under
WiFi TX step, UART edges 65ns vs the 104us bit budget, relay driver deep
saturation (Vce 68.6mV) with flyback contained, and the power-loss ordering
proven (ESP32 in brownout-reset before contacts transfer). The one modeled
mid-frame relay-gap sag confirms the firmware's inter-frame-gap switching
mitigation is mandatory (already in PLAN.md), not a defect.

Revalidation clean sweep: 132/132 host parser tests, 8816 KV pairs replayed
from real logic-analyzer captures with 0 desyncs, verbatim ESP-IDF esp32s3
build + stable QEMU boot, all 31 BOM C-numbers live-in-stock (>=3x) with the
new 330R part (C23138), and both enclosure STLs render 2-manifold in
OpenSCAD (now committed for direct JLC3DP upload).

Adversarial order gate re-ran every load-bearing check independently and
returned GO: 14 machine-verified facts vs 4 bench-only items (rail noise,
BLE range, relay lifetime, motor byte-pacing), each mapped to its
firmware/PLAN.md treadmill-contact gate. REPORT cost table reconciled to the
13 live-confirmed Extended lines (~$77-107 all-in). Adds ORDER-READY.md
(click-by-click order steps + GO verdict) and VALIDATION.md round-2.

Co-Authored-By: Claude Fable 5 <noreply@anthropic.com>
Claude-Session: https://claude.ai/code/session_01Gopx84MbomUJwTr592YXHN
Parts:
- D5, D6, D7: value PESD3V3L1BA -> PESD3V3L1BA-N; LCSC C51450 -> C316020
- LED1: value GREEN-0603 -> XL-1608UGC-04; LCSC C72043 -> C965804
- R11: value 1k -> 330R; LCSC C21190 -> C23138
- R12: value 2k -> 1k; LCSC C22975 -> C21190
