File: hardware/Esp32Tap/kicad/Esp32Tap.kicad_sch (KiCad schematic)
At the start: 50 parts, among them J1 RJ45_Console_54602-908LF, J2 RJ45_Motor_54602-908LF, J3 USB-C_HRO_TYPE-C-31-M-12, K1 G6K-2F-Y-TR DC3, Q1 S8050, SW1 KMR2-EN, SW2 KMR2-BOOT, U1 ESP32-S3-WROOM-1-N8, U2 TPS54202DDCR, U3 USBLC6-2SC6

Commit message: feat(hardware): generate typed rev B schematic
Parts:
- removed D2: SS34, Diode_SMD:D_SMA, symbol esp32tap:SYM_D2
- added C12: 56pF C0G 0603, Capacitor_SMD:C_0603_1608Metric, symbol esp32tap:SYM_C12
- added C13: DNP, Capacitor_SMD:C_0603_1608Metric, symbol esp32tap:SYM_C13
- added C14: DNP, Capacitor_SMD:C_0603_1608Metric, symbol esp32tap:SYM_C14
- added C15: 1uF/25V X7R 0603, Capacitor_SMD:C_0603_1608Metric, symbol esp32tap:SYM_C15
- added C16: 4.7uF/25V X7R 0805, Capacitor_SMD:C_0805_2012Metric, symbol esp32tap:SYM_C16
- added C17: 100nF, Capacitor_SMD:C_0603_1608Metric, symbol esp32tap:SYM_C17
- added C18: 1nF/50V C0G 0603, Capacitor_SMD:C_0603_1608Metric, symbol esp32tap:SYM_C18
- added C19: 1nF/50V C0G 0603, Capacitor_SMD:C_0603_1608Metric, symbol esp32tap:SYM_C19
- added C20: 100nF, Capacitor_SMD:C_0603_1608Metric, symbol esp32tap:SYM_C20
- added C21: 100nF, Capacitor_SMD:C_0603_1608Metric, symbol esp32tap:SYM_C21
- added Q2: 2N7002, Package_TO_SOT_SMD:SOT-23, symbol esp32tap:SYM_Q2
- added R15: 22R, Resistor_SMD:R_0603_1608Metric, symbol esp32tap:SYM_R15
- added R16: 22R, Resistor_SMD:R_0603_1608Metric, symbol esp32tap:SYM_R16
- added R17: 150k, Resistor_SMD:R_0603_1608Metric, symbol esp32tap:SYM_R17
- added R18: 10k, Resistor_SMD:R_0603_1608Metric, symbol esp32tap:SYM_R18
- added R19: 255k, Resistor_SMD:R_0603_1608Metric, symbol esp32tap:SYM_R19
- added R20: 10k, Resistor_SMD:R_0603_1608Metric, symbol esp32tap:SYM_R20
- added R21: 10k, Resistor_SMD:R_0603_1608Metric, symbol esp32tap:SYM_R21
- added R22: 100k, Resistor_SMD:R_0603_1608Metric, symbol esp32tap:SYM_R22
- added R23: 10k, Resistor_SMD:R_0603_1608Metric, symbol esp32tap:SYM_R23
- added R24: 10k, Resistor_SMD:R_0603_1608Metric, symbol esp32tap:SYM_R24
- added R25: 10k, Resistor_SMD:R_0603_1608Metric, symbol esp32tap:SYM_R25
- added R26: 10k, Resistor_SMD:R_0603_1608Metric, symbol esp32tap:SYM_R26
- added R27: 10k, Resistor_SMD:R_0603_1608Metric, symbol esp32tap:SYM_R27
- added R28: 10k, Resistor_SMD:R_0603_1608Metric, symbol esp32tap:SYM_R28
- added R29: 10k, Resistor_SMD:R_0603_1608Metric, symbol esp32tap:SYM_R29
- added R30: 10k, Resistor_SMD:R_0603_1608Metric, symbol esp32tap:SYM_R30
- added R31: 10k, Resistor_SMD:R_0603_1608Metric, symbol esp32tap:SYM_R31
- added TP10: TX_GATE, TestPoint:TestPoint_Pad_1.5x1.5mm, symbol esp32tap:SYM_TP10
- added TP11: TX_DRV, TestPoint:TestPoint_Pad_1.5x1.5mm, symbol esp32tap:SYM_TP11
- added TP12: K1_NC_FB, TestPoint:TestPoint_Pad_1.5x1.5mm, symbol esp32tap:SYM_TP12
- added TP13: K1_NO_FB, TestPoint:TestPoint_Pad_1.5x1.5mm, symbol esp32tap:SYM_TP13
- added TP5: VIN, TestPoint:TestPoint_Pad_1.5x1.5mm, symbol esp32tap:SYM_TP5
- added TP6: +5V_RLY, TestPoint:TestPoint_Pad_1.5x1.5mm, symbol esp32tap:SYM_TP6
- added TP7: TREAD_OK, TestPoint:TestPoint_Pad_1.5x1.5mm, symbol esp32tap:SYM_TP7
- added TP8: RELAY_GATE, TestPoint:TestPoint_Pad_1.5x1.5mm, symbol esp32tap:SYM_TP8
- added TP9: RELAY_SW, TestPoint:TestPoint_Pad_1.5x1.5mm, symbol esp32tap:SYM_TP9
- added U4: TPS3700DDCR, Package_TO_SOT_SMD:SOT-23-6, symbol esp32tap:SYM_U4
- added U5: TPS70950DBVR, Package_TO_SOT_SMD:SOT-23-5, symbol esp32tap:SYM_U5
- added U6: SN74LVC2G08DCTR, Package_SO:SSOP-8_2.95x2.8mm_P0.65mm, symbol esp32tap:SYM_U6
- added U7: SN74LVC1G126DBVR, Package_TO_SOT_SMD:SOT-23-5, symbol esp32tap:SYM_U7
- C1, SW1, SW2: JLC Class (none) -> Extended; Unit Cost USD (none) -> 0.100
- C10: JLC Class (none) -> Basic; Unit Cost USD (none) -> 0.006
- C11: value 1uF -> 100nF; JLC Class (none) -> Basic; LCSC C15849 -> C14663; Unit Cost USD (none) -> 0.004
- C2, C3: value 4.7uF/50V X7R 1206 -> 10uF/25V X7R 1206; JLC Class (none) -> Basic; LCSC C29823 -> C14860; Unit Cost USD (none) -> 0.040
- C4, C5, C9: JLC Class (none) -> Basic; Unit Cost USD (none) -> 0.004
- C6, C7: value 22uF/16V 0805 -> 22uF/25V X7R 1210; footprint Capacitor_SMD:C_0805_2012Metric -> Capacitor_SMD:C_1210_3225Metric; JLC Class (none) -> Extended; LCSC C45783 -> C2918511; Unit Cost USD (none) -> 0.080
- C8: JLC Class (none) -> Basic; Unit Cost USD (none) -> 0.010
- D1: JLC Class (none) -> Basic; Unit Cost USD (none) -> 0.050
- D3: value SMBJ12A -> SMBJ10A; JLC Class (none) -> Extended; LCSC C151251 -> C151250; Unit Cost USD (none) -> 0.050
- D4: value 1N4148WS -> SMAJ6.0CA; footprint Diode_SMD:D_SOD-323 -> Diode_SMD:D_SMA; JLC Class (none) -> Extended; LCSC C2128 -> C80275; Unit Cost USD (none) -> 0.050
- D5, D6, D7: JLC Class (none) -> Extended; Unit Cost USD (none) -> 0.061
- F1: value PolyFuse 0.75A/16V 1206L075/16WR -> 1812L075/24DR; footprint Fuse:Fuse_1206_3216Metric -> Fuse:Fuse_1812_4532Metric; JLC Class (none) -> Extended; LCSC C371166 -> C207065; Unit Cost USD (none) -> 0.100
- J1, J2: JLC Class (none) -> Extended-THT; Unit Cost USD (none) -> 0.380
- J3: JLC Class (none) -> Extended; Unit Cost USD (none) -> 0.160
- K1: value G6K-2F-Y-TR DC3 -> G6K-2F-Y-TR DC5; JLC Class (none) -> Extended; LCSC C2153097 -> C47190; Unit Cost USD (none) -> 1.500
- L1: JLC Class (none) -> Extended; Unit Cost USD (none) -> 0.070
- LED1: JLC Class (none) -> Extended; Unit Cost USD (none) -> 0.005
- LED2: JLC Class (none) -> Basic; Unit Cost USD (none) -> 0.020
- Q1: value S8050 -> BC817-40,215; JLC Class (none) -> Extended; LCSC C2146 -> C52801; Unit Cost USD (none) -> 0.030
- R1, R10, R11, R12, R13, R14, R2, R3, R4, R5, R6, R9: JLC Class (none) -> Basic; Unit Cost USD (none) -> 0.002
- R7, R8: value 4.7k -> 10k; JLC Class (none) -> Basic; LCSC C23162 -> C25804; Unit Cost USD (none) -> 0.002
- TP1, TP2, TP3, TP4: JLC Class (none) -> none; Unit Cost USD (none) -> 0.000
- U1: JLC Class (none) -> Extended; Unit Cost USD (none) -> 3.200
- U2: JLC Class (none) -> Extended; Unit Cost USD (none) -> 0.350
- U3: JLC Class (none) -> Extended; Unit Cost USD (none) -> 0.200
Connections:
- net +3V3: now also C12.1, C20.1, C21.1, R21.1, R25.1, R26.1, R30.1, R31.1, U6.8 (VCC), U7.5 (VCC); no longer D4.1 (K), K1.1 (COIL+)
- net +8V_F: no longer C1.1 (+), C2.1, D3.1 (K)
- net CONS6: no longer K1.7 (NC_B)
- net ESP_TX: now also U7.2 (A); no longer R6.1
- net FB: now also C12.2
- net GND: now also K1.6 (COM_B), C13.2, C14.2, C15.2, C16.2, C17.2, C18.2, C19.2, C20.2, C21.2, Q2.2 (S), R18.2, R20.2, R22.2, R23.2, R24.2, R27.2, R28.2, R29.2, U4.2 (GND), U5.2 (GND), U6.4 (GND), U7.3 (GND)
- net IO0: now also R31.2
- net MOT6: no longer K1.6 (COM_B)
- net RELAY_SW: now also TP9.1
- net TX_DRV: now also TP11.1; no longer K1.5 (NO_B)
- net USB_DN_MCU: now also R15.1; no longer U1.13 (IO19/USB_D-)
- net USB_DP_MCU: now also R16.1; no longer U1.14 (IO20/USB_D+)
- net VBUS: now also Q2.1 (G), R29.1
- net VIN: now also C1.1 (+), C2.1, D3.1 (K), C15.1, C17.1, R17.1, R19.1, TP5.1, U4.5 (VDD), U5.1 (IN)
- net K1_NC_FB: now reaches U1.4 (IO4)
- net K1_NC_FB: now also K1.7 (NC_B), R25.2, TP12.1
- net K1_NO_FB: now reaches U1.5 (IO5)
- net K1_NO_FB: now also K1.5 (NO_B), R26.2, TP13.1
- net TREAD_OK: now reaches U1.6 (IO6)
- net TREAD_OK: now also R21.2, R22.1, TP7.1, U4.1 (OUTA), U4.6 (OUTB), U6.2 (1B), U6.6 (2B)
- net VBUS_PRESENT_N: now reaches U1.7 (IO7)
- net VBUS_PRESENT_N: now also Q2.3 (D), R30.2
- net TX_ENABLE: now reaches U1.8 (IO15)
- net TX_ENABLE: now also R27.1, U6.5 (2A)
- net RELAY_EN renamed RELAY_CMD
- net RELAY_CMD: now also R23.1, U6.1 (1A); no longer R9.1
- new net +5V_RLY: C16.1, D4.1 (K), K1.1 (COIL+), TP6.1, U5.5 (OUT)
- new net OV_SENSE: C19.1, R19.2, R20.1, U4.4 (INB-)
- new net RELAY_GATE: R24.1, R9.1, TP8.1, U5.3 (EN), U6.7 (1Y)
- new net TX_BUF: R6.1, U7.4 (Y)
- new net TX_GATE: R28.1, TP10.1, U6.3 (2Y), U7.1 (OE)
- new net USB_DN_R: C13.1, R15.2, U1.13 (IO19/USB_D-)
- new net USB_DP_R: C14.1, R16.2, U1.14 (IO20/USB_D+)
- new net UV_SENSE: C18.1, R17.2, R18.1, U4.3 (INA+)
- no-connect marks 28 -> 24
Other:
- title: Esp32Tap - ESP32-S3 Precor serial-bus tap -> Esp32Tap Rev B - ESP32-S3 Precor serial-bus tap

Commit message: fix(hardware): harden Rev B artifact generation
Parts:
- C13, C14, TP1, TP10, TP11, TP12, TP13, TP2, TP3, TP4, TP5, TP6, TP7, TP8, TP9: now left out of the parts list

Commit message: hardware: generate validated Esp32Tap Rev B PCB
Parts:
- C12, C15, C16, C18, C19, C2, C3, R19: JLC Class Basic -> Extended
- R9: value 1k -> 560R; LCSC C21190 -> C23204
Changed lines of the file:
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@@
     (exclude_from_sim no) (in_bom yes) (on_board yes) (dnp no)
     (property "Reference" "R9" (at 192.50 240.84 0) (effects (font (size 1.27 1.27)) (justify left)))
-    (property "Value" "1k" (at 192.50 254.46 0) (effects (font (size 1.27 1.27)) (justify left)))
+    (property "Value" "560R" (at 192.50 254.46 0) (effects (font (size 1.27 1.27)) (justify left)))
     (property "Footprint" "Resistor_SMD:R_0603_1608Metric" (at 190.50 247.65 0) (effects (font (size 1.27 1.27)) (hide yes)))
     (property "Datasheet" "" (at 190.50 247.65 0) (effects (font (size 1.27 1.27)) (hide yes)))
-    (property "LCSC" "C21190" (at 190.50 247.65 0) (effects (font (size 1.27 1.27)) (hide yes)))
+    (property "LCSC" "C23204" (at 190.50 247.65 0) (effects (font (size 1.27 1.27)) (hide yes)))
     (property "JLC Class" "Basic" (at 190.50 247.65 0) (effects (font (size 1.27 1.27)) (hide yes)))
     (property "Unit Cost USD" "0.002" (at 190.50 247.65 0) (effects (font (size 1.27 1.27)) (hide yes)))
-    (property "Description" "Relay driver base resistor" (at 190.50 247.65 0) (effects (font (size 1.27 1.27)) (hide yes)))
+    (property "Description" "Relay driver base resistor (forced beta <= 10 at conservative drive)" (at 190.50 247.65 0) (effects (font (size 1.27 1.27)) (hide yes)))
     (pin "1")
     (pin "2")
@@
     (property "Datasheet" "" (at 190.50 521.97 0) (effects (font (size 1.27 1.27)) (hide yes)))
     (property "LCSC" "C23354" (at 190.50 521.97 0) (effects (font (size 1.27 1.27)) (hide yes)))
-    (property "JLC Class" "Basic" (at 190.50 521.97 0) (effects (font (size 1.27 1.27)) (hide yes)))
+    (property "JLC Class" "Extended" (at 190.50 521.97 0) (effects (font (size 1.27 1.27)) (hide yes)))
     (property "Unit Cost USD" "0.002" (at 190.50 521.97 0) (effects (font (size 1.27 1.27)) (hide yes)))
     (property "Description" "Overvoltage-sense divider top, 1%" (at 190.50 521.97 0) (effects (font (size 1.27 1.27)) (hide yes)))
@@
     (property "Datasheet" "" (at 264.16 430.53 0) (effects (font (size 1.27 1.27)) (hide yes)))
     (property "LCSC" "C14860" (at 264.16 430.53 0) (effects (font (size 1.27 1.27)) (hide yes)))
-    (property "JLC Class" "Basic" (at 264.16 430.53 0) (effects (font (size 1.27 1.27)) (hide yes)))
+    (property "JLC Class" "Extended" (at 264.16 430.53 0) (effects (font (size 1.27 1.27)) (hide yes)))
     (property "Unit Cost USD" "0.040" (at 264.16 430.53 0) (effects (font (size 1.27 1.27)) (hide yes)))
     (property "Description" "Input ceramic" (at 264.16 430.53 0) (effects (font (size 1.27 1.27)) (hide yes)))
@@
     (property "Datasheet" "" (at 264.16 461.01 0) (effects (font (size 1.27 1.27)) (hide yes)))
     (property "LCSC" "C14860" (at 264.16 461.01 0) (effects (font (size 1.27 1.27)) (hide yes)))
-    (property "JLC Class" "Basic" (at 264.16 461.01 0) (effects (font (size 1.27 1.27)) (hide yes)))
+    (property "JLC Class" "Extended" (at 264.16 461.01 0) (effects (font (size 1.27 1.27)) (hide yes)))
     (property "Unit Cost USD" "0.040" (at 264.16 461.01 0) (effects (font (size 1.27 1.27)) (hide yes)))
     (property "Description" "Buck VIN ceramic (at pin)" (at 264.16 461.01 0) (effects (font (size 1.27 1.27)) (hide yes)))
@@
     (property "Datasheet" "" (at 340.36 217.17 0) (effects (font (size 1.27 1.27)) (hide yes)))
     (property "LCSC" "C39148" (at 340.36 217.17 0) (effects (font (size 1.27 1.27)) (hide yes)))
-    (property "JLC Class" "Basic" (at 340.36 217.17 0) (effects (font (size 1.27 1.27)) (hide yes)))
+    (property "JLC Class" "Extended" (at 340.36 217.17 0) (effects (font (size 1.27 1.27)) (hide yes)))
     (property "Unit Cost USD" "0.004" (at 340.36 217.17 0) (effects (font (size 1.27 1.27)) (hide yes)))
     (property "Description" "Buck feed-forward capacitor directly across R1" (at 340.36 217.17 0) (effects (font (size 1.27 1.27)) (hide yes)))
@@
     (property "Datasheet" "" (at 340.36 308.61 0) (effects (font (size 1.27 1.27)) (hide yes)))
     (property "LCSC" "C106858" (at 340.36 308.61 0) (effects (font (size 1.27 1.27)) (hide yes)))
-    (property "JLC Class" "Basic" (at 340.36 308.61 0) (effects (font (size 1.27 1.27)) (hide yes)))
+    (property "JLC Class" "Extended" (at 340.36 308.61 0) (effects (font (size 1.27 1.27)) (hide yes)))
     (property "Unit Cost USD" "0.010" (at 340.36 308.61 0) (effects (font (size 1.27 1.27)) (hide yes)))
     (property "Description" "U5 input bypass" (at 340.36 308.61 0) (effects (font (size 1.27 1.27)) (hide yes)))
@@
     (property "Datasheet" "" (at 340.36 339.09 0) (effects (font (size 1.27 1.27)) (hide yes)))
     (property "LCSC" "C354262" (at 340.36 339.09 0) (effects (font (size 1.27 1.27)) (hide yes)))
-    (property "JLC Class" "Basic" (at 340.36 339.09 0) (effects (font (size 1.27 1.27)) (hide yes)))
+    (property "JLC Class" "Extended" (at 340.36 339.09 0) (effects (font (size 1.27 1.27)) (hide yes)))
     (property "Unit Cost USD" "0.020" (at 340.36 339.09 0) (effects (font (size 1.27 1.27)) (hide yes)))
     (property "Description" "U5 relay-supply output capacitor" (at 340.36 339.09 0) (effects (font (size 1.27 1.27)) (hide yes)))
@@
     (property "Datasheet" "" (at 340.36 400.05 0) (effects (font (size 1.27 1.27)) (hide yes)))
     (property "LCSC" "C342541" (at 340.36 400.05 0) (effects (font (size 1.27 1.27)) (hide yes)))
-    (property "JLC Class" "Basic" (at 340.36 400.05 0) (effects (font (size 1.27 1.27)) (hide yes)))
+    (property "JLC Class" "Extended" (at 340.36 400.05 0) (effects (font (size 1.27 1.27)) (hide yes)))
     (property "Unit Cost USD" "0.004" (at 340.36 400.05 0) (effects (font (size 1.27 1.27)) (hide yes)))
     (property "Description" "Undervoltage-sense filter" (at 340.36 400.05 0) (effects (font (size 1.27 1.27)) (hide yes)))
@@
     (property "Datasheet" "" (at 340.36 430.53 0) (effects (font (size 1.27 1.27)) (hide yes)))
     (property "LCSC" "C342541" (at 340.36 430.53 0) (effects (font (size 1.27 1.27)) (hide yes)))
-    (property "JLC Class" "Basic" (at 340.36 430.53 0) (effects (font (size 1.27 1.27)) (hide yes)))
+    (property "JLC Class" "Extended" (at 340.36 430.53 0) (effects (font (size 1.27 1.27)) (hide yes)))
     (property "Unit Cost USD" "0.004" (at 340.36 430.53 0) (effects (font (size 1.27 1.27)) (hide yes)))
     (property "Description" "Overvoltage-sense filter" (at 340.36 430.53 0) (effects (font (size 1.27 1.27)) (hide yes)))

Commit message: hardware: redesign Esp32Tap as compact turnkey Rev C (#52)
Redesign the serial-powered Esp32Tap around compact SMT Micro-Fit harness interfaces, regenerate and validate the PCB/enclosure/manufacturing package, and add fail-closed evidence, ngspice, vendor, and handoff documentation.

The hardware remains HOLD pending live JLC process/quote confirmation and physical installed measurements.
Parts:
- J1: value RJ45_Console_54602-908LF -> 430450809; footprint Connector_RJ:RJ45_Amphenol_54602-x08_Horizontal -> Connector_Molex:Molex_Micro-Fit_3.0_43045-0809_2x04-1MP_P3.00mm_Horizontal; JLC Class Extended-THT -> Extended; LCSC C2847314 -> C240838; Unit Cost USD 0.380 -> 2.140
- J2: value RJ45_Motor_54602-908LF -> 430451010; footprint Connector_RJ:RJ45_Amphenol_54602-x08_Horizontal -> Connector_Molex:Molex_Micro-Fit_3.0_43045-1010_2x05-1MP_P3.00mm_Horizontal; JLC Class Extended-THT -> Extended; LCSC C2847314 -> C563827; Unit Cost USD 0.380 -> 2.580
- SW1: value KMR2-EN -> SKRPACE010; footprint Button_Switch_SMD:SW_Push_1P1T_NO_CK_KMR2 -> Button_Switch_SMD:SW_SPST_SKRPACE010; LCSC C72443 -> C139797; Unit Cost USD 0.100 -> 0.060
- SW2: value KMR2-BOOT -> SKRPACE010; footprint Button_Switch_SMD:SW_Push_1P1T_NO_CK_KMR2 -> Button_Switch_SMD:SW_SPST_SKRPACE010; LCSC C72443 -> C139797; Unit Cost USD 0.100 -> 0.060
Connections:
- no-connect marks 24 -> 26
Other:
- title: Esp32Tap Rev B - ESP32-S3 Precor serial-bus tap -> Esp32Tap Rev C - ESP32-S3 Precor serial-bus tap
