File: hardware/Esp32Tap/kicad/Esp32Tap.kicad_sch (KiCad schematic)
At the start: 90 parts, among them J1 430450809, J2 430451010, J3 USB-C_HRO_TYPE-C-31-M-12, K1 G6K-2F-Y-TR DC5, Q1 BC817-40,215, Q2 2N7002, SW1 SKRPACE010, SW2 SKRPACE010, U1 ESP32-S3-WROOM-1-N8, U2 TPS54202DDCR, U3 USBLC6-2SC6, U4 TPS3700DDCR, U5 TPS70950DBVR, U6 SN74LVC2G08DCTR, U7 SN74LVC1G126DBVR

Commit message: hardware(Esp32Tap): add TREAD_OK series R32 + move C1 to in-stock 1210 ceramic
Two generator-driven fixes on top of the merged Rev C, both regenerated and
gate-green (make check: 744 tests, byte-reproducible artifacts, ngspice,
enclosure, fab audit, JLC stock).

- R32 (4.7k, C23162): series isolation between the TREAD_OK window-comparator
  node and ESP32 IO6. Prevents a misconfigured GPIO from overriding the U4
  voltage window or contending with its open-drain output (review finding B2).
  Splits net TREAD_OK -> TREAD_OK_MCU. Also hardens gen_pcb via_allowed() to
  check clearance on all copper layers, not just F.Cu (pre-existing latent bug).

- C1: 100uF/25V SMD electrolytic (C72477, CP_Elec_6.3x7.7) -> 22uF/25V X7R
  1210 ceramic (C2918511, same part as C6/C7). JLC had no in-stock electrolytic
  for that footprint; the ceramic is non-polarized, machine-placeable, and
  reuses an existing footprint. Reduces input bulk (acceptable: buck already
  has ceramic front-end caps); revisit value for production hold-up.

Verified on JLCPCB: all 75 parts place on Standard PCBA (J1/J2 Micro-Fit
C240838/C563827 confirmed, U1 -> N8R2 C2913204).

Note: a global lint hook black-reformatted the touched .py files, inflating the
diff; the functional change is the R32 net/part edits and the C1 part/footprint swap.

Co-Authored-By: Claude Opus 4.8 <noreply@anthropic.com>
Claude-Session: https://claude.ai/code/session_01Gopx84MbomUJwTr592YXHN
Parts:
- added R32: 4.7k, Resistor_SMD:R_0603_1608Metric, symbol esp32tap:SYM_R32
- C1: value 100uF/25V -> 22uF/25V X7R 1210; footprint Capacitor_SMD:CP_Elec_6.3x7.7 -> Capacitor_SMD:C_1210_3225Metric; LCSC C72477 -> C2918511; Unit Cost USD 0.100 -> 0.080
Connections:
- net TREAD_OK: now also R32.1; no longer U1.6 (IO6)
- new net TREAD_OK_MCU: R32.2, U1.6 (IO6)
Other:
- moved on the sheet: C1, C10, C11, C12, C13, C14, C15, C16, C17, C18, C19, C2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

Commit message: hardware(Esp32Tap): Rev D — on-board right-angle SMD RJ45, delete pigtails
Replace the Rev C Micro-Fit headers + external RJ45 pigtails with two
on-board, edge-mounted, right-angle SMD RJ45 jacks. Fully machine-assembled
by JLC (SMT), cheaper than Rev C, and eliminates the custom-cable line item.

- J1/J2: Molex 0441440003 (LCSC C585890) — unshielded 8P8C, right-angle,
  SMD, JLC "SMT Assembly", in stock. Edge-mounted with the mating opening
  facing off the board edge so a standard RJ45 plug reaches through the
  enclosure wall aperture. Verified right-angle by rendering the real 3D
  model (JLC's catalog "Mounting Type" field is unreliable for RJ45).
- Deleted hardware/Esp32Tap/harness/ (both pigtails, housings, terminals).
- Reused the Rev B RJ45 1:1 pinout (pin1/7 GND, 2/8 +8V, 3-6 data/serial).
- Enclosure: RJ45 wall apertures replace the Micro-Fit cutouts.
- Preserved unchanged: R32 (TREAD_OK series resistor), C1 (22uF 1210
  ceramic), ESP32-S3-N8R2, relay, buck, all other nets/parts.
- Bumped board revision C -> D (silkscreen, title block, validators, docs).

Tradeoff: the two jacks are the identical part, so the Rev C Micro-Fit
mechanical console/motor anti-swap keying is gone; CONSOLE/MOTOR silkscreen
(+ optional jack color) is the differentiator now.

make check green: 640 tests, byte-reproducible artifacts, ngspice (8 decks
x3, host+docker), enclosure validator, fab audit, JLC stock. DRC 0.

Note: a global lint hook black-reformats touched .py files, inflating the
diff; the functional change is the connector swap + harness deletion + rev bump.

Co-Authored-By: Claude Opus 4.8 (1M context) <noreply@anthropic.com>
Claude-Session: https://claude.ai/code/session_01Gopx84MbomUJwTr592YXHN
Parts:
- J1: value 430450809 -> 441440003; footprint Connector_Molex:Molex_Micro-Fit_3.0_43045-0809_2x04-1MP_P3.00mm_Horizontal -> RJ45_SMD:RJ45-SMD_441440003; LCSC C240838 -> C585890; Unit Cost USD 2.140 -> 0.350
- J2: value 430451010 -> 441440003; footprint Connector_Molex:Molex_Micro-Fit_3.0_43045-1010_2x05-1MP_P3.00mm_Horizontal -> RJ45_SMD:RJ45-SMD_441440003; LCSC C563827 -> C585890; Unit Cost USD 2.580 -> 0.350
Connections:
- no-connect marks 26 -> 28
Other:
- title: Esp32Tap Rev C - ESP32-S3 Precor serial-bus tap -> Esp32Tap Rev D - ESP32-S3 Precor serial-bus tap
- moved on the sheet: C1, C10, C11, C12, C13, C14, C15, C16, C17, C18, C19, C2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

Commit message: hardware(Esp32Tap): Rev E layout — J2 (MOTOR) to right short edge, USB-C to bottom edge
J1 (CONSOLE) stays on the left short edge; J2 mirrors it on the right so the
board reads console-to-motor left to right. USB-C cluster (J3/U3) relocates to
the bottom edge with fully re-authored F.Cu-only matched pair (skew 0.08 mm).
Full-board +8V trunk with In1 GND mesh; router now blocks footprint-embedded
rule areas (ESP32-S3 antenna keepout) on all routing layers. All gates green:
clean-check byte-reproducible, 640 pytest, sims, DRC/ERC 0, enclosure re-cut
with one RJ45 aperture per short wall.

Known open items (next commit): RJ45 mating faces are 180° reversed (latent
Rev D bug), jacks not yet Y-aligned, silkscreen still says rev D.

Co-Authored-By: Claude Fable 5 <noreply@anthropic.com>
Claude-Session: https://claude.ai/code/session_017aRNAWKnAHt47TQVDu1G6J
Other:
- title: Esp32Tap Rev D - ESP32-S3 Precor serial-bus tap -> Esp32Tap Rev E - ESP32-S3 Precor serial-bus tap
Changed lines of the file:
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@@
 (kicad_sch (version 20231120) (generator "esp32tap_gen")
   (paper "A1")
-  (title_block (title "Esp32Tap Rev D - ESP32-S3 Precor serial-bus tap") (date "2026-07-24") (rev "D") (company "precor-9.3x") (comment 1 "Status: generated Rev D typed schematic") (comment 2 "Source of truth: tools/design.py") (comment 3 "Generated by tools/gen_sch.py; do not hand-edit"))
+  (title_block (title "Esp32Tap Rev E - ESP32-S3 Precor serial-bus tap") (date "2026-07-24") (rev "E") (company "precor-9.3x") (comment 1 "Status: generated Rev E typed schematic") (comment 2 "Source of truth: tools/design.py") (comment 3 "Generated by tools/gen_sch.py; do not hand-edit"))
   (symbol (lib_id "esp32tap:SYM_J1") (at 40.64 44.45 0) (unit 1)
     (exclude_from_sim no) (in_bom yes) (on_board yes) (dnp no)
